File: Pinky/Pinky.kicad_pcb (KiCad board)
At the start: 2 copper layers, 142.4 x 120.7 mm, 74 parts, among them J1 MJ-4PP-9, J2 i2c-pin, J3 i2c-pin, J4 LED, SW1 RESET_SW, SW10 SW_PUSH, SW11 SW_PUSH, SW12 SW_PUSH, SW13 SW_PUSH, SW14 SW_PUSH, SW15 SW_PUSH, SW16 SW_PUSH, SW17 SW_PUSH, SW18 SW_PUSH, SW19 SW_PUSH, SW2 SW_PUSH, SW20 SW_PUSH, SW21 SW_PUSH, SW22 SW_PUSH, SW23 SW_PUSH, SW24 SW_PUSH, SW25 SW_PUSH, SW26 SW_PUSH, SW27 SW_PUSH, SW28 SW_PUSH, SW29 SW_PUSH, SW3 SW_PUSH, SW30 SW_PUSH, SW31 SW_PUSH, SW32 SW_PUSH, SW33 SW_PUSH, SW4 SW_PUSH, SW5 SW_PUSH, SW6 SW_PUSH, SW7 SW_PUSH, SW8 SW_PUSH, SW9 SW_PUSH, U1 ProMicro

Commit message: [WIP] wiring & layouting
Parts:
- added Ref**: Val**, kbd:HOLE, F.Cu at (59.5, 59.5)
- added Ref**: Val**, kbd:HOLE, F.Cu at (59.5, 97.6)
- added Ref**: Val**, kbd:HOLE, F.Cu at (153.3, 119.1)
- added Ref**: Val**, kbd:HOLE, F.Cu at (117.3, 95.7)
- added Ref**: Val**, kbd:HOLE, F.Cu at (155.4, 84.2)
- moved Ref** 18.9 mm to (117.3, 57.6)
- moved JP1 2.80 mm to (74.1, 129.7)
- moved D30 2.00 mm to (162.3, 103.9)
- moved J4 1.53 mm to (156.2, 105.5)
- moved P2 0.10 mm to (81.7, 123.3)
- moved J1 0.10 mm to (180.5, 112.2)
- renumbered J2 to P1, J3 to P2
Routing:
- net VCC: track 0.00 -> 170.3 mm, vias 0 -> 1
- net col0: track 0.00 -> 161.6 mm, vias 0 -> 5
- net row0: track 0.00 -> 102.9 mm, vias 0 -> 4
- net row1: track 0.00 -> 81.5 mm, vias 0 -> 2
- net row2: track 0.00 -> 61.8 mm
- net Net-(D1-Pad2): track 0.00 -> 33.3 mm, vias 0 -> 2
- net Net-(D3-Pad2): track 0.00 -> 32.9 mm, vias 0 -> 2
- net Net-(D2-Pad2): track 0.00 -> 32.6 mm, vias 0 -> 3
Other:
- board size 142.4 x 120.7 mm -> 142.2 x 120.4 mm

Commit message: [WIP] wiring & layouting
Routing:
- net Net-(D4-Pad2): track 0.00 -> 23.4 mm, vias 0 -> 2

Commit message: [WIP] wiring & layouting
Parts:
- SW10, SW11, SW12, SW13, SW14, SW15, SW16, SW17, SW19, SW2, SW20, SW21, SW22, SW24, SW25, SW26, SW27, SW29, SW3, SW30, SW31, SW32, SW4, SW5, SW6, SW7, SW8, SW9: footprint kbd:CherryMX_KailhLowProfile_Hotswap -> kbd:CherryMX_Hotswap
- moved SW17 1.03 mm to (107.8, 100.6)
- moved SW13 0.88 mm to (87.2, 105.1)
- moved SW32 0.64 mm to (167.4, 120.0), turned to 0 degrees
- moved SW21 0.54 mm to (126.7, 85.9)
- moved SW9 0.44 mm to (68.7, 107.4)
- moved SW8 0.40 mm to (69.5, 88.2)
- moved SW7 0.40 mm to (68.7, 69.2)
- moved SW4 0.36 mm to (50.2, 88.4)
- moved SW27 0.35 mm to (145.0, 108.8)
- moved SW19 0.34 mm to (125.9, 47.9)
- moved SW11 0.33 mm to (87.8, 67.2)
- moved SW15 0.30 mm to (106.9, 63.2)
- moved SW20 0.30 mm to (126.5, 67.2)
- moved SW31 0.25 mm to (164.5, 93.6)
- moved SW25 0.25 mm to (145.4, 70.8)
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Routing:
- net col0: track 161.6 -> 0.00 mm, vias 5 -> 0
- net row0: track 102.9 -> 0.00 mm, vias 4 -> 0
- net row1: track 81.5 -> 0.29 mm, vias 2 -> 0
- net row2: track 61.8 -> 0.00 mm
- net Net-(D1-Pad2): track 33.3 -> 0.35 mm, vias 2 -> 0
- net Net-(D3-Pad2): track 32.9 -> 0.00 mm, vias 2 -> 0
- net Net-(D2-Pad2): track 32.6 -> 0.72 mm, vias 3 -> 0
- net Net-(D4-Pad2): track 23.4 -> 0.00 mm, vias 2 -> 0

Commit message: [WIP] layout completed
Parts:
- moved JP1 12.3 mm to (77.2, 117.8)
- moved P1 11.2 mm to (92.4, 123.5)
- moved P2 11.2 mm to (92.4, 126.7)
- moved R1 11.2 mm to (87.3, 123.5)
- moved R2 11.2 mm to (87.3, 126.7)
- moved SW1 11.2 mm to (88.9, 132.6)
- moved U1 2.83 mm to (59.3, 125.8)
- moved SW17 1.03 mm to (107.2, 101.4)
- moved SW13 0.88 mm to (88.1, 105.2)
- moved SW32 0.65 mm to (166.8, 119.8), turned to 337 degrees
- moved SW21 0.54 mm to (126.2, 86.2)
- moved SW9 0.44 mm to (69.0, 107.2)
- moved SW8 0.40 mm to (69.0, 88.1)
- moved SW7 0.40 mm to (69.0, 69.0)
- moved SW4 0.36 mm to (50.0, 88.1)
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Routing:
- net VCC: track 170.3 -> 15.6 mm, vias 1 -> 0
Other:
- outline, holes or cut-outs redrawn

Commit message: [WIP] layout completed
Routing:
- net col0: track 0.00 -> 77.1 mm, vias 0 -> 1
- net Net-(D1-Pad2): track 0.35 -> 31.7 mm, vias 0 -> 1
Other:
- outline, holes or cut-outs redrawn
Changed lines of the file:
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@@
     (thickness 1.6)
     (drawings 150)
-    (tracks 11)
+    (tracks 34)
     (zones 0)
     (modules 79)
@@
   (gr_line (start 155 146.7) (end 170.5 155.6) (layer Edge.Cuts) (width 0.2))
   (gr_line (start 137 140) (end 153.9 146.2) (layer Edge.Cuts) (width 0.2))
-  (gr_line (start 117.5 136.3) (end 135.4 139.5) (layer Edge.Cuts) (width 0.2))
+  (gr_line (start 117.5 136.3) (end 135.3 139.5) (layer Edge.Cuts) (width 0.2))
   (gr_line (start 179.8 140.9) (end 171.5 155.4) (layer Edge.Cuts) (width 0.2))
   (gr_line (start 171.5 135.2) (end 179.5 139.8) (layer Edge.Cuts) (width 0.2))
@@
   (segment (start 170.198266 110.10853) (end 166.6 110.10853) (width 0.5) (layer F.Cu) (net 35))
   (segment (start 156.2 105.5) (end 156.299994 105.5) (width 0.5) (layer B.Cu) (net 35))
+  (segment (start 54.568001 52.325001) (end 54.5 52.325001) (width 0.25) (layer F.Cu) (net 41))
+  (segment (start 57 49.893002) (end 54.568001 52.325001) (width 0.25) (layer F.Cu) (net 41))
+  (segment (start 57 47.42) (end 57 49.893002) (width 0.25) (layer F.Cu) (net 41))
+  (via (at 54.5 52.325001) (size 0.8) (drill 0.4) (layers F.Cu B.Cu) (net 41))
+  (segment (start 43 48.67) (end 43 47.42) (width 0.25) (layer B.Cu) (net 41))
+  (segment (start 43 49.893002) (end 43 48.67) (width 0.25) (layer B.Cu) (net 41))
+  (segment (start 43.074999 52.325001) (end 43 52.4) (width 0.25) (layer B.Cu) (net 41))
+  (segment (start 54.5 52.325001) (end 43.074999 52.325001) (width 0.25) (layer B.Cu) (net 41))
+  (segment (start 43 52.4) (end 43 66.47) (width 0.25) (layer B.Cu) (net 41))
+  (segment (start 43 47.42) (end 43 52.4) (width 0.25) (layer B.Cu) (net 41))
+  (segment (start 43 67.72) (end 43 104.57) (width 0.25) (layer B.Cu) (net 41))
+  (segment (start 43 66.47) (end 43 67.72) (width 0.25) (layer B.Cu) (net 41))
   (segment (start 51.575 60) (end 51.4 60) (width 0.25) (layer F.Cu) (net 42))
   (segment (start 51.2 60) (end 51.375 60) (width 0.25) (layer F.Cu) (net 42))
+  (segment (start 55.7 43.63) (end 54.47 42.4) (width 0.25) (layer B.Cu) (net 42))
+  (segment (start 55.7 44.88) (end 55.7 43.63) (width 0.25) (layer B.Cu) (net 42))
+  (segment (start 54.47 42.4) (end 54.47 42.4) (width 0.25) (layer B.Cu) (net 42))
+  (via (at 54.47 42.4) (size 0.8) (drill 0.4) (layers F.Cu B.Cu) (net 42))
+  (segment (start 44.3 43.63) (end 44.3 44.88) (width 0.25) (layer F.Cu) (net 42))
+  (segment (start 45.53 42.4) (end 44.3 43.63) (width 0.25) (layer F.Cu) (net 42))
+  (segment (start 54.47 42.4) (end 45.53 42.4) (width 0.25) (layer F.Cu) (net 42))
+  (segment (start 56.305001 46.735001) (end 55.7 46.13) (width 0.25) (layer B.Cu) (net 42))
+  (segment (start 56.305001 57.504999) (end 56.305001 46.735001) (width 0.25) (layer B.Cu) (net 42))
+  (segment (start 55.7 46.13) (end 55.7 44.88) (width 0.25) (layer B.Cu) (net 42))
+  (segment (start 53.81 60) (end 56.305001 57.504999) (width 0.25) (layer B.Cu) (net 42))
   (segment (start 51.775 78.325) (end 51.775 79.05) (width 0.25) (layer F.Cu) (net 43))
 )

Commit message: [WIP] wiring
Parts:
- moved D4 39.6 mm to (50.0, 111.0)
- moved D8 20.6 mm to (69.0, 111.0)
- moved D12 6.22 mm to (88.1, 109.0)
- moved JP1 4.20 mm to (77.2, 122.0)
- moved Ref** 4.02 mm to (116.0, 53.8)
- moved Ref** 4.02 mm to (116.0, 91.9)
- moved Ref** 3.92 mm to (154.1, 80.5)
- moved Ref** 1.32 mm to (154.6, 119.3)
Routing:
- net row0: track 0.29 -> 204.5 mm
- net col3: track 0.00 -> 181.4 mm, vias 0 -> 6
- net row1: track 0.00 -> 181.2 mm, vias 0 -> 2
- net row2: track 0.00 -> 180.3 mm
- net col4: track 0.00 -> 162.4 mm, vias 0 -> 6
- net col2: track 0.00 -> 158.7 mm, vias 0 -> 4
- net col5: track 0.00 -> 150.3 mm, vias 0 -> 4
- net col1: track 0.00 -> 149.7 mm, vias 0 -> 4
- net col6: track 0.00 -> 115.8 mm, vias 0 -> 3
- net col0: track 77.1 -> 144.0 mm, vias 1 -> 4
- net Net-(D16-Pad2): track 0.00 -> 35.6 mm, vias 0 -> 1
- net Net-(D17-Pad2): track 0.00 -> 35.4 mm, vias 0 -> 3
- net Net-(D21-Pad2): track 0.00 -> 35.2 mm, vias 0 -> 1
- net Net-(D30-Pad2): track 0.00 -> 34.9 mm, vias 0 -> 1
- net Net-(D7-Pad2): track 0.00 -> 34.0 mm, vias 0 -> 1
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Other:
- board size 142.2 x 120.4 mm -> 142.2 x 120.5 mm

Commit message: [WIP] wiring
Parts:
- moved D4 39.9 mm to (88.6, 121.2)
- moved D8 20.8 mm to (88.6, 118.2)
- moved JP1 10.1 mm to (77.7, 132.1)
- moved D12 6.22 mm to (88.6, 115.2)
- moved R1 3.02 mm to (87.3, 126.5)
- moved P1 3.00 mm to (92.4, 126.5)
- moved P2 3.00 mm to (92.4, 129.7)
- moved R2 3.00 mm to (87.3, 129.7)
- moved SW1 1.00 mm to (88.9, 133.6)
- moved J4 0.82 mm to (155.4, 105.7)
Routing:
- net Net-(J1-PadA): track 0.00 -> 96.3 mm, vias 0 -> 4
- net col4: track 162.4 -> 236.8 mm, vias 6 -> 9
- net row3: track 22.4 -> 94.7 mm
- net col6: track 115.8 -> 184.9 mm, vias 3 -> 6
- net row4: track 0.00 -> 63.7 mm
- net Net-(D32-Pad2): track 0.00 -> 41.5 mm, vias 0 -> 3
- net col3: track 181.4 -> 221.7 mm
- net Net-(D27-Pad2): track 0.00 -> 36.3 mm, vias 0 -> 3
- net col5: track 150.3 -> 185.0 mm, vias 4 -> 6
- net Net-(D22-Pad2): track 0.00 -> 34.3 mm, vias 0 -> 3
- net Net-(D4-Pad2): track 28.3 -> 61.8 mm, vias 2 -> 4
- net Net-(D31-Pad2): track 0.00 -> 31.9 mm, vias 0 -> 1
- net Net-(D26-Pad2): track 15.0 -> 36.7 mm
- net Net-(D12-Pad2): track 17.8 -> 33.7 mm
- net Net-(D8-Pad2): track 28.3 -> 43.7 mm
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
Commit message: [WIP] wiring
Parts:
- moved D4 44.8 mm to (50.0, 98.4)
- moved D8 27.8 mm to (69.1, 98.4)
- moved D31 24.5 mm to (162.4, 104.2), turned to 0 degrees
- moved D16 22.6 mm to (107.1, 92.6)
- moved D26 21.6 mm to (145.2, 100.2), turned to 0 degrees
- moved D21 20.9 mm to (126.1, 96.5), turned to 0 degrees
- moved D12 18.6 mm to (88.1, 96.6)
- moved J4 12.2 mm to (154.9, 93.5)
- moved D30 2.90 mm to (164.3, 101.8)
- moved D11 2.00 mm to (88.1, 94.2)
- moved D15 2.00 mm to (107.2, 90.4)
- moved D20 2.00 mm to (126.2, 94.2)
- moved D25 2.00 mm to (145.2, 98.0)
- moved D3 1.97 mm to (50.0, 96.1)
- moved D7 1.97 mm to (69.0, 96.1)
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Routing:
- net row0: track 204.5 -> 159.4 mm
- net Net-(D1-Pad2): track 34.3 -> 18.0 mm
- net col0: track 144.0 -> 131.2 mm
- net col1: track 149.7 -> 141.5 mm, vias 4 -> 3
- net Net-(D5-Pad2): track 33.9 -> 27.4 mm
