File: Pinky/Pinky.sch (KiCad schematic (older format))
At the start: 73 parts, among them J1 MJ-4PP-9, J2 i2c-pin, J3 i2c-pin, J4 LED, SW1 RESET_SW, SW10 SW_PUSH, SW11 SW_PUSH, SW12 SW_PUSH, SW13 SW_PUSH, SW14 SW_PUSH, SW15 SW_PUSH, SW16 SW_PUSH, SW17 SW_PUSH, SW18 SW_PUSH, SW19 SW_PUSH, SW2 SW_PUSH, SW20 SW_PUSH, SW21 SW_PUSH, SW22 SW_PUSH, SW23 SW_PUSH, SW24 SW_PUSH, SW25 SW_PUSH, SW26 SW_PUSH, SW27 SW_PUSH, SW28 SW_PUSH, SW29 SW_PUSH, SW3 SW_PUSH, SW30 SW_PUSH, SW31 SW_PUSH, SW32 SW_PUSH, SW33 SW_PUSH, SW4 SW_PUSH, SW5 SW_PUSH, SW6 SW_PUSH, SW7 SW_PUSH, SW8 SW_PUSH, SW9 SW_PUSH, U1 ProMicro

Commit message: [WIP] wiring & layouting
Parts:
- renumbered J2 to P1, J3 to P2
Changed lines of the file:
@@
 EESchema Schematic File Version 4
-LIBS:petit_split-cache
+LIBS:Pinky-cache
 EELAYER 26 0
 EELAYER END
@@
 $EndComp
 $Comp
-L Connector_Generic:Conn_01x01 J2
+L Connector_Generic:Conn_01x01 P1
 U 1 1 5BFC5069
 P 2375 3320
-F 0 "J2" V 2341 3232 50  0000 R CNN
+F 0 "P1" V 2341 3232 50  0000 R CNN
 F 1 "i2c-pin" V 2475 3450 50  0000 R CNN
 F 2 "kbd:1pin_conn" H 2375 3320 50  0001 C CNN
@@
 	1855 3670 2375 3670
 $Comp
-L Connector_Generic:Conn_01x01 J3
+L Connector_Generic:Conn_01x01 P2
 U 1 1 5BFDAF4C
 P 2375 3870
-F 0 "J3" V 2248 3950 50  0000 L CNN
+F 0 "P2" V 2248 3950 50  0000 L CNN
 F 1 "i2c-pin" V 2339 3950 50  0000 L CNN
 F 2 "kbd:1pin_conn" H 2375 3870 50  0001 C CNN

Commit message: [WIP] wiring & layouting
Parts:
- SW10, SW11, SW12, SW13, SW14, SW15, SW16, SW17, SW19, SW2, SW20, SW21, SW22, SW24, SW25, SW26, SW27, SW29, SW3, SW30, SW31, SW32, SW4, SW5, SW6, SW7, SW8, SW9: footprint kbd:CherryMX_KailhLowProfile_Hotswap -> kbd:CherryMX_Hotswap
Changed lines of the file:
@@
 F 0 "SW2" H 4920 3125 50  0000 C CNN
 F 1 "SW_PUSH" H 4920 3034 50  0000 C CNN
-F 2 "kbd:CherryMX_KailhLowProfile_Hotswap" H 4920 2870 50  0001 C CNN
+F 2 "kbd:CherryMX_Hotswap" H 4920 2870 50  0001 C CNN
 F 3 "" H 4920 2870 50  0000 C CNN
 	1    4920 2870
@@
 F 0 "SW6" H 5840 3125 50  0000 C CNN
 F 1 "SW_PUSH" H 5840 3034 50  0000 C CNN
-F 2 "kbd:CherryMX_KailhLowProfile_Hotswap" H 5840 2870 50  0001 C CNN
+F 2 "kbd:CherryMX_Hotswap" H 5840 2870 50  0001 C CNN
 F 3 "" H 5840 2870 50  0000 C CNN
 	1    5840 2870
@@
 F 0 "SW7" H 5840 3825 50  0000 C CNN
 F 1 "SW_PUSH" H 5840 3734 50  0000 C CNN
-F 2 "kbd:CherryMX_KailhLowProfile_Hotswap" H 5840 3570 50  0001 C CNN
+F 2 "kbd:CherryMX_Hotswap" H 5840 3570 50  0001 C CNN
 F 3 "" H 5840 3570 50  0000 C CNN
 	1    5840 3570
@@
 F 0 "SW4" H 4920 4485 50  0000 C CNN
 F 1 "SW_PUSH" H 4920 4394 50  0000 C CNN
-F 2 "kbd:CherryMX_KailhLowProfile_Hotswap" H 4920 4230 50  0001 C CNN
+F 2 "kbd:CherryMX_Hotswap" H 4920 4230 50  0001 C CNN
 F 3 "" H 4920 4230 50  0000 C CNN
 	1    4920 4230
@@
 F 0 "SW5" H 4920 5165 50  0000 C CNN
 F 1 "SW_PUSH" H 4920 5074 50  0000 C CNN
-F 2 "kbd:CherryMX_KailhLowProfile_Hotswap" H 4920 4910 50  0001 C CNN
+F 2 "kbd:CherryMX_Hotswap" H 4920 4910 50  0001 C CNN
 F 3 "" H 4920 4910 50  0000 C CNN
 	1    4920 4910
@@
 F 0 "SW8" H 5840 4485 50  0000 C CNN
 F 1 "SW_PUSH" H 5840 4394 50  0000 C CNN
-F 2 "kbd:CherryMX_KailhLowProfile_Hotswap" H 5840 4230 50  0001 C CNN
+F 2 "kbd:CherryMX_Hotswap" H 5840 4230 50  0001 C CNN
 F 3 "" H 5840 4230 50  0000 C CNN
 	1    5840 4230
@@
 F 0 "SW9" H 5840 5165 50  0000 C CNN
 F 1 "SW_PUSH" H 5840 5074 50  0000 C CNN
-F 2 "kbd:CherryMX_KailhLowProfile_Hotswap" H 5840 4910 50  0001 C CNN
+F 2 "kbd:CherryMX_Hotswap" H 5840 4910 50  0001 C CNN
 F 3 "" H 5840 4910 50  0000 C CNN
 	1    5840 4910
@@
 F 0 "SW3" H 4920 3825 50  0000 C CNN
 F 1 "SW_PUSH" H 4920 3734 50  0000 C CNN
-F 2 "kbd:CherryMX_KailhLowProfile_Hotswap" H 4920 3570 50  0001 C CNN
+F 2 "kbd:CherryMX_Hotswap" H 4920 3570 50  0001 C CNN
 F 3 "" H 4920 3570 50  0000 C CNN
 	1    4920 3570
@@
 F 0 "SW10" H 6730 3125 50  0000 C CNN
 F 1 "SW_PUSH" H 6730 3034 50  0000 C CNN
-F 2 "kbd:CherryMX_KailhLowProfile_Hotswap" H 6730 2870 50  0001 C CNN
+F 2 "kbd:CherryMX_Hotswap" H 6730 2870 50  0001 C CNN
 F 3 "" H 6730 2870 50  0000 C CNN
 	1    6730 2870
@@
 F 0 "SW11" H 6730 3825 50  0000 C CNN
 F 1 "SW_PUSH" H 6730 3734 50  0000 C CNN
-F 2 "kbd:CherryMX_KailhLowProfile_Hotswap" H 6730 3570 50  0001 C CNN
+F 2 "kbd:CherryMX_Hotswap" H 6730 3570 50  0001 C CNN
 F 3 "" H 6730 3570 50  0000 C CNN
 	1    6730 3570
@@
 F 0 "SW14" H 7605 3125 50  0000 C CNN
 F 1 "SW_PUSH" H 7605 3034 50  0000 C CNN
-F 2 "kbd:CherryMX_KailhLowProfile_Hotswap" H 7605 2870 50  0001 C CNN
+F 2 "kbd:CherryMX_Hotswap" H 7605 2870 50  0001 C CNN
 F 3 "" H 7605 2870 50  0000 C CNN
 	1    7605 2870
@@
 F 0 "SW15" H 7605 3825 50  0000 C CNN
 F 1 "SW_PUSH" H 7605 3734 50  0000 C CNN
-F 2 "kbd:CherryMX_KailhLowProfile_Hotswap" H 7605 3570 50  0001 C CNN
+F 2 "kbd:CherryMX_Hotswap" H 7605 3570 50  0001 C CNN
 F 3 "" H 7605 3570 50  0000 C CNN
 	1    7605 3570
@@
 F 0 "SW12" H 6730 4485 50  0000 C CNN
 F 1 "SW_PUSH" H 6730 4394 50  0000 C CNN
-F 2 "kbd:CherryMX_KailhLowProfile_Hotswap" H 6730 4230 50  0001 C CNN
+F 2 "kbd:CherryMX_Hotswap" H 6730 4230 50  0001 C CNN
 F 3 "" H 6730 4230 50  0000 C CNN
 	1    6730 4230
@@
 F 0 "SW16" H 7605 4485 50  0000 C CNN
 F 1 "SW_PUSH" H 7605 4394 50  0000 C CNN
-F 2 "kbd:CherryMX_KailhLowProfile_Hotswap" H 7605 4230 50  0001 C CNN
+F 2 "kbd:CherryMX_Hotswap" H 7605 4230 50  0001 C CNN
 F 3 "" H 7605 4230 50  0000 C CNN
 	1    7605 4230
@@
 F 0 "SW13" H 6730 5165 50  0000 C CNN
 F 1 "SW_PUSH" H 6730 5074 50  0000 C CNN
-F 2 "kbd:CherryMX_KailhLowProfile_Hotswap" H 6730 4910 50  0001 C CNN
+F 2 "kbd:CherryMX_Hotswap" H 6730 4910 50  0001 C CNN
 F 3 "" H 6730 4910 50  0000 C CNN
 	1    6730 4910
@@
 F 0 "SW17" H 7605 5165 50  0000 C CNN
 F 1 "SW_PUSH" H 7605 5074 50  0000 C CNN
-F 2 "kbd:CherryMX_KailhLowProfile_Hotswap" H 7605 4910 50  0001 C CNN
+F 2 "kbd:CherryMX_Hotswap" H 7605 4910 50  0001 C CNN
 F 3 "" H 7605 4910 50  0000 C CNN
 	1    7605 4910
@@
 F 0 "SW19" H 8460 3125 50  0000 C CNN
 F 1 "SW_PUSH" H 8460 3034 50  0000 C CNN
-F 2 "kbd:CherryMX_KailhLowProfile_Hotswap" H 8460 2870 50  0001 C CNN
+F 2 "kbd:CherryMX_Hotswap" H 8460 2870 50  0001 C CNN
 F 3 "" H 8460 2870 50  0000 C CNN
 	1    8460 2870
@@
 F 0 "SW20" H 8460 3825 50  0000 C CNN
 F 1 "SW_PUSH" H 8460 3734 50  0000 C CNN
-F 2 "kbd:CherryMX_KailhLowProfile_Hotswap" H 8460 3570 50  0001 C CNN
+F 2 "kbd:CherryMX_Hotswap" H 8460 3570 50  0001 C CNN
 F 3 "" H 8460 3570 50  0000 C CNN
 	1    8460 3570
@@
 F 0 "SW21" H 8460 4485 50  0000 C CNN
 F 1 "SW_PUSH" H 8460 4394 50  0000 C CNN
-F 2 "kbd:CherryMX_KailhLowProfile_Hotswap" H 8460 4230 50  0001 C CNN
+F 2 "kbd:CherryMX_Hotswap" H 8460 4230 50  0001 C CNN
 F 3 "" H 8460 4230 50  0000 C CNN
 	1    8460 4230
@@
 F 0 "SW22" H 8460 5165 50  0000 C CNN
 F 1 "SW_PUSH" H 8460 5074 50  0000 C CNN
-F 2 "kbd:CherryMX_KailhLowProfile_Hotswap" H 8460 4910 50  0001 C CNN
+F 2 "kbd:CherryMX_Hotswap" H 8460 4910 50  0001 C CNN
 F 3 "" H 8460 4910 50  0000 C CNN
 	1    8460 4910
@@
 F 0 "SW24" H 9300 3125 50  0000 C CNN
 F 1 "SW_PUSH" H 9300 3034 50  0000 C CNN
-F 2 "kbd:CherryMX_KailhLowProfile_Hotswap" H 9300 2870 50  0001 C CNN
+F 2 "kbd:CherryMX_Hotswap" H 9300 2870 50  0001 C CNN
 F 3 "" H 9300 2870 50  0000 C CNN
 	1    9300 2870
@@
 F 0 "SW25" H 9300 3825 50  0000 C CNN
 F 1 "SW_PUSH" H 9300 3734 50  0000 C CNN
-F 2 "kbd:CherryMX_KailhLowProfile_Hotswap" H 9300 3570 50  0001 C CNN
+F 2 "kbd:CherryMX_Hotswap" H 9300 3570 50  0001 C CNN
 F 3 "" H 9300 3570 50  0000 C CNN
 	1    9300 3570
@@
 F 0 "SW26" H 9300 4485 50  0000 C CNN
 F 1 "SW_PUSH" H 9300 4394 50  0000 C CNN
-F 2 "kbd:CherryMX_KailhLowProfile_Hotswap" H 9300 4230 50  0001 C CNN
+F 2 "kbd:CherryMX_Hotswap" H 9300 4230 50  0001 C CNN
 F 3 "" H 9300 4230 50  0000 C CNN
 	1    9300 4230
@@
 F 0 "SW27" H 9300 5165 50  0000 C CNN
 F 1 "SW_PUSH" H 9300 5074 50  0000 C CNN
-F 2 "kbd:CherryMX_KailhLowProfile_Hotswap" H 9300 4910 50  0001 C CNN
+F 2 "kbd:CherryMX_Hotswap" H 9300 4910 50  0001 C CNN
 F 3 "" H 9300 4910 50  0000 C CNN
 	1    9300 4910
@@
 F 0 "SW29" H 10185 3125 50  0000 C CNN
 F 1 "SW_PUSH" H 10185 3034 50  0000 C CNN
-F 2 "kbd:CherryMX_KailhLowProfile_Hotswap" H 10185 2870 50  0001 C CNN
+F 2 "kbd:CherryMX_Hotswap" H 10185 2870 50  0001 C CNN
 F 3 "" H 10185 2870 50  0000 C CNN
 	1    10185 2870
@@
 F 0 "SW30" H 10185 3825 50  0000 C CNN
 F 1 "SW_PUSH" H 10185 3734 50  0000 C CNN
-F 2 "kbd:CherryMX_KailhLowProfile_Hotswap" H 10185 3570 50  0001 C CNN
+F 2 "kbd:CherryMX_Hotswap" H 10185 3570 50  0001 C CNN
 F 3 "" H 10185 3570 50  0000 C CNN
 	1    10185 3570
@@
 F 0 "SW31" H 10185 4485 50  0000 C CNN
 F 1 "SW_PUSH" H 10185 4394 50  0000 C CNN
-F 2 "kbd:CherryMX_KailhLowProfile_Hotswap" H 10185 4230 50  0001 C CNN
+F 2 "kbd:CherryMX_Hotswap" H 10185 4230 50  0001 C CNN
 F 3 "" H 10185 4230 50  0000 C CNN
 	1    10185 4230
@@
 F 0 "SW32" H 10185 5165 50  0000 C CNN
 F 1 "SW_PUSH" H 10185 5074 50  0000 C CNN
-F 2 "kbd:CherryMX_KailhLowProfile_Hotswap" H 10185 4910 50  0001 C CNN
+F 2 "kbd:CherryMX_Hotswap" H 10185 4910 50  0001 C CNN
 F 3 "" H 10185 4910 50  0000 C CNN
 	1    10185 4910

Commit message: finished wiring
Parts:
- removed J4: LED, kbd:StripLED_rev, symbol Connector_Generic:Conn_01x03
Connections:
- net led: no longer names the net of U1.1 (TX)
- no-connect marks 3 -> 4
Changed lines of the file:
@@
 Wire Wire Line
 	2375 3670 2380 3670
-Text GLabel 1205 1445 0    50   Input ~ 0
-led
-$Comp
-L Connector_Generic:Conn_01x03 J4
-U 1 1 5BE2F8C9
-P 1680 5905
-F 0 "J4" H 1600 5580 50  0000 C CNN
-F 1 "LED" H 1600 5671 50  0000 C CNN
-F 2 "kbd:StripLED_rev" H 1680 5905 50  0001 C CNN
-F 3 "~" H 1680 5905 50  0001 C CNN
-	1    1680 5905
-	-1   0    0    1
-$EndComp
-Text GLabel 1880 5905 2    50   Input ~ 0
-led
-$Comp
-L power:GND #PWR010
-U 1 1 5BE3304A
-P 1880 6005
-F 0 "#PWR010" H 1880 5755 50  0001 C CNN
-F 1 "GND" H 1885 5832 50  0000 C CNN
-F 2 "" H 1880 6005 50  0001 C CNN
-F 3 "" H 1880 6005 50  0001 C CNN
-	1    1880 6005
-	1    0    0    -1
-$EndComp
-$Comp
-L power:VCC #PWR09
-U 1 1 5BE339D9
-P 1880 5805
-F 0 "#PWR09" H 1880 5655 50  0001 C CNN
-F 1 "VCC" H 1897 5978 50  0000 C CNN
-F 2 "" H 1880 5805 50  0001 C CNN
-F 3 "" H 1880 5805 50  0001 C CNN
-	1    1880 5805
-	1    0    0    -1
-$EndComp
 Text GLabel 1205 1845 0    50   Input ~ 0
 sda
@@
 	1    0    0    -1
 $EndComp
+NoConn ~ 1205 1445
 $EndSCHEMATC
