File: pcb/Pinky4.kicad_pcb (KiCad board)
At the start: 2 copper layers, 139 x 120 mm, 80 parts, among them J1 MJ-4PP-9, P1 i2c-pin, P2 i2c-pin, SW1 RESET_SW, SW10 SW_PUSH, SW11 SW_PUSH, SW12 SW_PUSH, SW13 SW_PUSH, SW14 SW_PUSH, SW15 SW_PUSH, SW16 SW_PUSH, SW17 SW_PUSH, SW18 SW_PUSH, SW19 SW_PUSH, SW2 SW_PUSH, SW20 SW_PUSH, SW21 SW_PUSH, SW22 SW_PUSH, SW23 SW_PUSH, SW24 SW_PUSH, SW25 SW_PUSH, SW26 SW_PUSH, SW27 SW_PUSH, SW28 SW_PUSH, SW29 SW_PUSH, SW3 SW_PUSH, SW30 SW_PUSH, SW31 SW_PUSH, SW32 SW_PUSH, SW33 SW_PUSH, SW4 SW_PUSH, SW5 SW_PUSH, SW6 SW_PUSH, SW7 SW_PUSH, SW8 SW_PUSH, SW9 SW_PUSH, U1 ProMicro

Commit message: jumper
Parts:
- JP1: value Jumper -> (none); footprint kbd:Jumper -> kbd:JPC2
Changed lines of the file:
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@@
-(kicad_pcb (version 20171130) (host pcbnew "(5.0.1-3-g963ef8bb5)")
+(kicad_pcb (version 20171130) (host pcbnew "(5.1.4-0-10_14)")
   (general
     (thickness 1.6)
@@
     (zone_45_only no)
     (trace_min 0.2)
-    (segment_width 0.15)
-    (edge_width 0.15)
     (via_size 0.6)
     (via_drill 0.4)
@@
     (uvia_min_size 0.4)
     (uvia_min_drill 0.3)
+    (edge_width 0.15)
+    (segment_width 0.15)
     (pcb_text_width 0.3)
     (pcb_text_size 1.5 1.5)
@@
     (add_net sda)
   )
+  (module kbd:JPC2 (layer F.Cu)
+    (at 81 133.8 90)
+    (attr smd)
+    (fp_text reference JP1 (at -2.413 0.127 90) (layer F.SilkS) hide
+      (effects (font (size 0.8128 0.8128) (thickness 0.1524)))
+    )
+    (fp_text value " " (at 1.9 0 -180) (layer F.SilkS)
+      (effects (font (size 0.8128 0.8128) (thickness 0.15)))
+    )
+    (fp_line (start -1.143 -0.889) (end 1.143 -0.889) (layer F.SilkS) (width 0.15))
+    (fp_line (start 1.143 -0.889) (end 1.143 0.889) (layer F.SilkS) (width 0.15))
+    (fp_line (start 1.143 0.889) (end -1.143 0.889) (layer F.SilkS) (width 0.15))
+    (fp_line (start -1.143 0.889) (end -1.143 -0.889) (layer F.SilkS) (width 0.15))
+    (pad 1 smd rect (at -0.50038 0 90) (size 0.635 1.143) (layers F.Cu F.Paste F.Mask)
+      (net 37 "Net-(J1-PadB)") (clearance 0.1905))
+    (pad 2 smd rect (at 0.50038 0 90) (size 0.635 1.143) (layers F.Cu F.Paste F.Mask)
+      (net 39 data) (clearance 0.1905))
+    (pad "" smd rect (at 0 0 180) (size 0.381 0.381) (layers F.Cu F.Paste F.Mask)
+      (clearance 0.00254))
+    (model smd\resistors\R0603.wrl
+      (offset (xyz 0 0 0.02539999961853028))
+      (scale (xyz 0.5 0.5 0.5))
+      (rotate (xyz 0 0 0))
+    )
+  )
   (module kbd:D3_TH_SMD (layer F.Cu)
     (at 128.9 121 350)
@@
       (rotate (xyz 0 0 0))
     )
-  )
-  (module kbd:Jumper (layer F.Cu)
-    (at 81 133.8 90)
-    (attr smd)
-    (fp_text reference JP1 (at -2.413 0.127 90) (layer F.SilkS) hide
-      (effects (font (size 0.8128 0.8128) (thickness 0.1524)))
-    )
-    (fp_text value Jumper (at 1.9 0 -180) (layer F.SilkS)
-      (effects (font (size 0.8128 0.8128) (thickness 0.15)))
-    )
-    (fp_line (start -1.143 -0.889) (end 1.143 -0.889) (layer F.SilkS) (width 0.15))
-    (fp_line (start 1.143 -0.889) (end 1.143 0.889) (layer F.SilkS) (width 0.15))
-    (fp_line (start 1.143 0.889) (end -1.143 0.889) (layer F.SilkS) (width 0.15))
-    (fp_line (start -1.143 0.889) (end -1.143 -0.889) (layer F.SilkS) (width 0.15))
-    (pad 1 smd rect (at -0.50038 0 90) (size 0.635 1.143) (layers F.Cu F.Paste F.Mask)
-      (net 37 "Net-(J1-PadB)") (clearance 0.1905))
-    (pad 2 smd rect (at 0.50038 0 90) (size 0.635 1.143) (layers F.Cu F.Paste F.Mask)
-      (net 39 data) (clearance 0.1905))
-    (model smd\resistors\R0603.wrl
-      (offset (xyz 0 0 0.02539999961853028))
-      (scale (xyz 0.5 0.5 0.5))
-      (rotate (xyz 0 0 0))
-    )
